Commit message: fixed mass in urdf

File: ros_ws/src/xela_description/xela_description/robot.urdf (robot description, URDF)
Before this commit: robot xela_description, 17 links, 16 joints
Links:
- link clipper: mass 0.00468118 -> 0.003
- link fingertop_unfied: mass 0.0384693 -> 0.016
- link fingertop_unfied_2: mass 0.0384693 -> 0.016
- link fingertop_unfied_3: mass 0.0384693 -> 0.016
- link leap_hand_xela_back_cover: mass 1.50836 -> 0.237
- link p2_unified: mass 0.0355531 -> 0.037
- link p2_unified_2: mass 0.0355531 -> 0.037
- link p2_unified_3: mass 0.0355531 -> 0.037
- link p3_unified: mass 0.0241611 -> 0.032
- link p3_unified_2: mass 0.0241611 -> 0.032
- link p3_unified_3: mass 0.0241611 -> 0.032
- link p4_unified: mass 0.0353104 -> 0.044
- link p4_unified_2: mass 0.0353104 -> 0.044
- link p4_unified_3: mass 0.0353104 -> 0.044
- link thfingertip_unified: mass 0.062548 -> 0.049
- link thp1_unified: mass 0.0325393 -> 0.038
- link thp2_unified: mass 0.0247742 -> 0.032
