Commit message: made xela_description urdf more consistant with leap_description

File: ros_ws/src/xela_description/urdf/finger.urdf (robot description, URDF)
Before this commit: robot xela_finger_generated, 5 links, 4 joints
Links:
- removed link rf_fingertop_unfied
- removed link rf_p2_unified
- removed link rf_p3_unified
- removed link rf_p4_unified
- added link rf_dip, mass 0.037; collision mesh filename=package://assets/p2_unified.stl; visual mesh filename=package://assets/p2_unified.stl
- added link rf_fingertip, mass 0.016; collision mesh filename=package://assets/fingertop_unfied.stl; visual mesh filename=package://assets/fingertop_unfied.stl
- added link rf_mcp, mass 0.044; collision mesh filename=package://assets/p4_unified.stl; visual mesh filename=package://assets/p4_unified.stl
- added link rf_pip, mass 0.032; collision mesh filename=package://assets/p3_unified.stl; visual mesh filename=package://assets/p3_unified.stl
- added link rf_realtip, mass 1e-06; collision sphere radius=0.005; visual sphere radius=0.005
Joints:
- added joint rf_realtip: type fixed, parent rf_fingertip, child rf_realtip, origin xyz=-0.02 -0.07 0.015 rpy=0.0 0.0 0.0, axis 0.0 0.0 -1.0
- joint base: child rf_p4_unified -> rf_mcp
- joint rf_dip: child rf_fingertop_unfied -> rf_fingertip; parent rf_p2_unified -> rf_dip
- joint rf_pip: child rf_p2_unified -> rf_dip; parent rf_p3_unified -> rf_pip
- joint rf_rot: child rf_p3_unified -> rf_pip; parent rf_p4_unified -> rf_mcp

File: ros_ws/src/xela_description/urdf/thumb.urdf (robot description, URDF)
Before this commit: robot xela_thumb_generated, 5 links, 4 joints
Links:
- removed link clipper
- removed link thfingertip_unified
- removed link thp1_unified
- removed link thp2_unified
- added link axl, mass 0.003; collision mesh filename=package://assets/clipper.stl; collision mesh filename=package://assets/thconnector.stl
- added link cmc, mass 0.032; collision mesh filename=package://assets/thp2_unified.stl; visual mesh filename=package://assets/thp2_unified.stl
- added link th_ipl, mass 0.049; collision mesh filename=package://assets/thfingertip_unified.stl; visual mesh filename=package://assets/thfingertip_unified.stl
- added link th_mcp, mass 0.038; collision mesh filename=package://assets/thp1_unified.stl; visual mesh filename=package://assets/thp1_unified.stl
Joints:
- joint base: child thp2_unified -> cmc
- joint th_axl: child clipper -> axl; parent thp2_unified -> cmc
- joint th_ipl: child thfingertip_unified -> th_ipl; parent thp1_unified -> th_mcp
- joint th_mcp: child thp1_unified -> th_mcp; parent clipper -> axl

Commit message: modyified keyboar d control a bit. wrote joint_config.json that contains joint limits

File: ros_ws/src/xela_description/urdf/finger.urdf (robot description, URDF)
Before this commit: robot xela_finger_generated, 6 links, 5 joints
Links:
- removed link rf_realtip
Joints:
- removed joint rf_realtip
- joint rf_dip: limit lower=-0.366519 upper=2.04204 effort=10 velocity=10 -> lower=-0.0873 upper=2.2689 effort=0.95 velocity=8.48
- joint rf_pip: limit lower=-0.506145 upper=1.88496 effort=10 velocity=10 -> lower=-0.262 upper=2.0944 effort=0.95 velocity=8.48
- joint rf_rot: limit lower=-1.0472 upper=1.0472 effort=10 velocity=10 -> lower=-0.349 upper=0.349 effort=0.95 velocity=8.48

File: ros_ws/src/xela_description/urdf/thumb.urdf (robot description, URDF)
Before this commit: robot xela_thumb_generated, 5 links, 4 joints
Joints:
- joint th_axl: limit lower=-0.349066 upper=2.0944 effort=10 velocity=10 -> lower=-0.305 upper=0.436 effort=0.95 velocity=8.48
- joint th_ipl: limit lower=-1.3439 upper=1.88496 effort=10 velocity=10 -> lower=-0.436 upper=1.309 effort=0.95 velocity=8.48
- joint th_mcp: limit lower=-0.471239 upper=2.44346 effort=10 velocity=10 -> lower=-0.262 upper=1.396 effort=0.95 velocity=8.48
