Commit message: created arm_server that alows for plan and execute action

File: ros_ws/src/multipanda_ros2/franka_moveit_config/srdf/panda_arm.xacro (robot description, xacro)
@@ -1,7 +1,9 @@
 <?xml version="1.0" ?>
 <robot xmlns:xacro="http://www.ros.org/wiki/xacro" name="panda">
-  <xacro:macro name="panda_arm" params="arm_id:='panda' ">
+  <xacro:macro name="panda_arm" params="arm_id:='panda' hand:=true">
     <xacro:include filename="$(find franka_moveit_config)/srdf/group_definition.xacro"/>
-    <xacro:group_definition arm_id="${arm_id}" group_name="${arm_id}_manipulator" tip_link="${arm_id}_hand_tcp"/>
+    <xacro:if value="${hand}">
+      <xacro:group_definition arm_id="${arm_id}" group_name="${arm_id}_manipulator" tip_link="${arm_id}_hand_tcp"/>
+    </xacro:if>
     <xacro:group_definition arm_id="${arm_id}" group_name="${arm_id}_arm" tip_link="${arm_id}_link8"/>
     <virtual_joint name="virtual_joint" type="fixed" parent_frame="world" child_link="${arm_id}_link0"/>
